File: Layout/keyboard.kicad_pcb (KiCad board)
At the start: 2 copper layers, 265.2 x 84.2 mm, 216 parts, among them J2 Conn_01x04_Socket, J3 Conn_01x04_Socket, J4 Conn_01x03_Socket, J5 Conn_01x03_Socket

Commit message: work done
Parts:
- removed the D_1 at (18.1, 11.0)
- removed the D_10 at (72.2, -10.5)
- removed the D_10 at (208.6, 10.0)
- removed the D_11 at (78.0, -40.7)
- removed the D_11 at (227.6, 10.0)
- removed the D_12 at (78.0, -37.3)
- removed the D_12 at (256.2, 10.0)
- removed the D_13 at (78.0, -34.0)
- removed the D_13 at (27.6, 29.1)
- removed D_14, D_15, D_16, D_17, D_18, D_19, D_20, D_21, D_22, D_23, D_24, D_25, D_26, D_27, D_28, D_29, D_30, D_31, D_32, D_33, D_34, D_35, D_36, D_37, D_38, D_39, D_40, D_41, D_42, D_43: D, Diode_SMD:D_SOD-123
- removed the D_2 at (72.2, -37.3)
- removed the D_2 at (56.1, 10.0)
- removed the D_3 at (72.2, -34.0)
- removed the D_3 at (75.2, 10.0)
- removed the D_4 at (72.2, -30.6)
- removed the D_4 at (94.2, 10.0)
- removed the D_5 at (72.2, -27.3)
- removed the D_5 at (113.3, 10.0)
- removed the D_6 at (72.2, -23.9)
- removed the D_6 at (132.3, 10.0)
- removed the D_7 at (72.2, -20.6)
- removed the D_7 at (151.4, 10.0)
- removed the D_8 at (72.2, -17.2)
- removed the D_8 at (170.4, 10.0)
- removed the D_9 at (72.2, -13.9)
- removed the D_9 at (189.5, 10.0)
- added D_10: D, Diode_SMD:D_SOD-123, F.Cu at (324.2, -18.0)
- added D_11: D, Diode_SMD:D_SOD-123, F.Cu at (324.2, -14.6)
- added D_12: D, Diode_SMD:D_SOD-123, F.Cu at (324.2, -11.3)
- added D_13: D, Diode_SMD:D_SOD-123, F.Cu at (324.2, -7.94)
- added D_2: D, Diode_SMD:D_SOD-123, F.Cu at (312.6, -18.0)
- added D_3: D, Diode_SMD:D_SOD-123, F.Cu at (312.6, -14.6)
- added D_4: D, Diode_SMD:D_SOD-123, F.Cu at (312.6, -11.3)
- added D_5: D, Diode_SMD:D_SOD-123, F.Cu at (312.6, -7.94)
- added D_6: D, Diode_SMD:D_SOD-123, F.Cu at (318.4, -18.0)
- added D_7: D, Diode_SMD:D_SOD-123, F.Cu at (318.4, -14.6)
- added D_8: D, Diode_SMD:D_SOD-123, F.Cu at (318.4, -11.3)
- added D_9: D, Diode_SMD:D_SOD-123, F.Cu at (318.4, -7.94)
- added J1: Conn_01x04_Socket, Connector_PinHeader_2.54mm:PinHeader_1x04_P2.54mm_Horizontal, F.Cu at (352.1, 25.0)
- added J6: Conn_01x03_Socket, Connector_PinHeader_2.54mm:PinHeader_1x03_P2.54mm_Horizontal, F.Cu at (352.1, 43.5)
- added J7: Conn_01x04_Socket, Connector_PinHeader_2.54mm:PinHeader_1x04_P2.54mm_Horizontal, F.Cu at (280.6, 38.1)
- added J8: Conn_01x03_Socket, Connector_PinHeader_2.54mm:PinHeader_1x03_P2.54mm_Horizontal, F.Cu at (280.6, 50.5)
- D_1, D_57, D_58, D_59, D_60, D_61, D_62, D_63, D_64, D_65, D_66, D_67, D_68, D_69, D_70, D_71, D_72, D_73, D_74, D_75, D_76, D_77, D_78, D_79, D_80, D_81, D_82, D_83, D_84, D_85, D_86, D_87, D_88, D_89, D_90, D_91, D_92, D_93, D_94, D_95, D_96, D_97, D_98: moved to B.Cu
- K_12: footprint MX_Solderable:MX-Solderable-1.5U -> MX_Solderable:MX-Solderable-1U
- K_13, K_5: footprint MX_Solderable:MX-Solderable-1.25U -> MX_Solderable:MX-Solderable-1U
- K_68: footprint Gateron_KS33_Solderable:Gateron-KS33-Solderable-1.5U -> Gateron_KS33_Solderable:Gateron-KS33-Solderable-1U
- U1: footprint JohnDeereLibrary:Waveshare_rp2040_Zero -> JohnDeereLibrary:Waveshare_rp2040_Tiny; moved to B.Cu
- moved K_65 289.6 mm to (318.4, 66.7)
- moved K_58 284.8 mm to (299.4, 9.53)
- moved K_61 276.1 mm to (299.4, 66.7)
- moved K_69 268.7 mm to (337.4, 66.7)
- moved K_68 268.1 mm to (337.4, 47.6)
- moved K_67 262.2 mm to (337.4, 28.6)
- moved K_60 254.6 mm to (299.4, 47.6)
- moved K_63 247.1 mm to (318.4, 28.6)
- moved K_66 241.5 mm to (337.4, 9.53)
- moved K_59 233.2 mm to (299.4, 28.6)
- moved K_62 226.1 mm to (318.4, 9.53)
- moved K_13 223.9 mm to (337.4, 66.7)
- moved K_5 223.2 mm to (299.4, 66.7)
- moved K_4 215.7 mm to (299.4, 47.6)
- moved K_3 208.3 mm to (299.4, 28.6)
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Routing:
- net row0: track 0.00 -> 353.1 mm
- net row1: track 0.00 -> 345.4 mm
- net row2: track 0.00 -> 315.0 mm
- net col11: track 0.00 -> 244.0 mm
- net col10: track 0.00 -> 229.0 mm
- net col12: track 0.00 -> 226.9 mm
- net col9: track 0.00 -> 217.7 mm
- net row3: track 0.00 -> 183.9 mm
- net col8: track 0.00 -> 181.5 mm
- net col7: track 0.00 -> 166.3 mm
- net col6: track 42.0 -> 150.9 mm
- net col0: track 88.1 -> 154.5 mm
- net col15: track 0.00 -> 56.4 mm
- net col14: track 0.00 -> 51.5 mm
- net col13: track 0.00 -> 48.1 mm
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
Commit message: Finish layout
Parts:
- D_10, D_11, D_12, D_13, D_2, D_3, D_4, D_5, D_6, D_7, D_8, D_9: moved to B.Cu
- J1, J2, J3, J7: footprint Connector_PinHeader_2.54mm:PinHeader_1x04_P2.54mm_Horizontal -> Connector_PinHeader_2.54mm:PinHeader_1x05_P2.54mm_Horizontal
- moved D_13 186.7 mm to (378.6, 170.7), turned to 90 degrees
- moved D_9 183.3 mm to (359.6, 170.7), turned to 90 degrees
- moved D_5 180.8 mm to (340.5, 170.7), turned to 90 degrees
- moved D_12 171.8 mm to (378.6, 151.6), turned to 90 degrees
- moved D_8 168.0 mm to (359.6, 151.6), turned to 90 degrees
- moved D_4 164.5 mm to (340.5, 150.8), turned to 90 degrees
- moved D_11 156.9 mm to (378.6, 132.6), turned to 90 degrees
- moved D_7 152.9 mm to (359.6, 132.6), turned to 90 degrees
- moved D_3 149.8 mm to (340.5, 132.6), turned to 90 degrees
- moved U1 146.0 mm to (200.7, 172.5)
- moved D_10 142.3 mm to (378.6, 113.5), turned to 90 degrees
- moved D_6 137.8 mm to (359.6, 113.5), turned to 90 degrees
- moved D_2 134.4 mm to (340.5, 113.5), turned to 90 degrees
- moved J5 130.0 mm to (45.2, 171.4)
- moved J4 129.9 mm to (306.8, 166.4)
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Connections:
- D_10 pad 1: Net-(D_10-K) -> row0
- D_11 pad 1: Net-(D_11-K) -> row1
- D_12 pad 1: Net-(D_12-K) -> row2
- D_13 pad 1: Net-(D_13-K) -> row3
- D_2 pad 1: Net-(D_10-K) -> row0
- D_3 pad 1: Net-(D_11-K) -> row1
- D_4 pad 1: Net-(D_12-K) -> row2
- D_5 pad 1: Net-(D_13-K) -> row3
- D_6 pad 1: Net-(D_10-K) -> row0
- D_7 pad 1: Net-(D_11-K) -> row1
- D_8 pad 1: Net-(D_12-K) -> row2
- D_9 pad 1: Net-(D_13-K) -> row3
- J1 pad 3: row2 -> unconnected-(J1-Pin_3-Pad3)
- J1 pad 4: row3 -> row2
- J2 pad 3: row2 -> unconnected-(J2-Pin_3-Pad3)
- J2 pad 4: row3 -> row2
- J3 pad 1: row0 -> row3
- J3 pad 2: row1 -> row2
- J3 pad 3: row2 -> unconnected-(J3-Pin_3-Pad3)
- J3 pad 4: row3 -> row1
- J4 pad 1: col7 -> col13
- J4 pad 2: col8 -> col14
- J4 pad 3: col9 -> col15
- J5 pad 1: col7 -> col15
- J5 pad 2: col8 -> col14
- J5 pad 3: col9 -> col13
- J6 pad 1: col7 -> col13
- J6 pad 2: col8 -> col14
- J6 pad 3: col9 -> col15
- J7 pad 1: row0 -> row3
- J7 pad 2: row1 -> row2
- J7 pad 3: row2 -> unconnected-(J7-Pin_3-Pad3)
- J7 pad 4: row3 -> row1
- J8 pad 1: col7 -> col15
- J8 pad 2: col8 -> col14
- J8 pad 3: col9 -> col13
Routing:
- net col14: track 51.5 -> 462.0 mm, vias 0 -> 2
- net row3: track 183.9 -> 592.5 mm
- net col15: track 56.4 -> 454.6 mm, vias 0 -> 1
- net col13: track 48.1 -> 445.2 mm, vias 0 -> 3
- net row2: track 315.0 -> 617.1 mm
- net row1: track 345.4 -> 567.4 mm, vias 0 -> 2
- net row0: track 353.1 -> 516.3 mm, vias 0 -> 2
- net col2: track 105.4 -> 169.4 mm
- net col0: track 154.5 -> 214.7 mm
- net col1: track 135.9 -> 194.7 mm
- net col7: track 166.3 -> 109.2 mm
- net col6: track 150.9 -> 94.8 mm
- net col8: track 181.5 -> 128.1 mm
- net col9: track 217.7 -> 168.4 mm
- net col3: track 104.3 -> 148.1 mm
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Other:
- board size 265.2 x 84.2 mm -> 340.5 x 86.5 mm
- board text added: "Pad side"
- board text added: "Pogo side"
- board text added: "V CUTS"

Commit message: Finished
Connections:
- U1 pad 22: (no net) -> unconnected-(U1-5v-Pad22)
Routing:
- net col2: track 169.4 -> 165.1 mm
- net col15: track 454.6 -> 452.3 mm
- net col5: track 126.0 -> 124.4 mm
- net col3: track 148.1 -> 146.5 mm
- net col4: track 136.4 -> 134.7 mm
- net col14: track 462.0 -> 463.3 mm
- net col13: track 445.2 -> 446.2 mm
- net col1: track 194.7 -> 193.8 mm
Other:
- outline, holes or cut-outs redrawn
