File: Layout/keyboard.kicad_sch (KiCad schematic)
At the start: 173 parts, among them J2 Conn_01x04_Socket, J3 Conn_01x04_Socket, J4 Conn_01x03_Socket, J5 Conn_01x03_Socket

Commit message: work done
Parts:
- added J1, J7: Conn_01x04_Socket, Connector_PinHeader_2.54mm:PinHeader_1x04_P2.54mm_Horizontal, symbol Connector:Conn_01x04_Socket
- added J6, J8: Conn_01x03_Socket, Connector_PinHeader_2.54mm:PinHeader_1x03_P2.54mm_Horizontal, symbol Connector:Conn_01x03_Socket
- K_12: footprint MX_Solderable:MX-Solderable-1.5U -> MX_Solderable:MX-Solderable-1U
- K_13, K_5: footprint MX_Solderable:MX-Solderable-1.25U -> MX_Solderable:MX-Solderable-1U
- K_68: footprint Gateron_KS33_Solderable:Gateron-KS33-Solderable-1.5U -> Gateron_KS33_Solderable:Gateron-KS33-Solderable-1U
- U1: footprint JohnDeereLibrary:Waveshare_rp2040_Zero -> JohnDeereLibrary:Waveshare_rp2040_Tiny
Connections:
- net col7: now also J6.1 (Pin_1), J8.1 (Pin_1)
- net col8: now also J6.2 (Pin_2), J8.2 (Pin_2)
- net col9: now also J6.3 (Pin_3), J8.3 (Pin_3)
- net row0: now also J1.1 (Pin_1), J7.1 (Pin_1); no longer D_10.1 (K), D_2.1 (K), D_6.1 (K)
- net row1: now also J1.2 (Pin_2), J7.2 (Pin_2); no longer D_11.1 (K), D_3.1 (K), D_7.1 (K)
- net row2: now also J1.3 (Pin_3), J7.3 (Pin_3); no longer D_12.1 (K), D_4.1 (K), D_8.1 (K)
- net row3: now also J1.4 (Pin_4), J7.4 (Pin_4); no longer D_13.1 (K), D_5.1 (K), D_9.1 (K)
- new net: D_11.1 (K), D_3.1 (K), D_7.1 (K)
- new net: D_10.1 (K), D_2.1 (K), D_6.1 (K)
- new net: D_13.1 (K), D_5.1 (K), D_9.1 (K)
- new net: D_12.1 (K), D_4.1 (K), D_8.1 (K)
Other:
- moved on the sheet: D_1, D_10, D_11, D_12, D_13, D_2, D_3, D_4, D_5, D_56, D_57, D_58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

Commit message: Finish layout
Parts:
- J1, J2, J3, J7: footprint Connector_PinHeader_2.54mm:PinHeader_1x04_P2.54mm_Horizontal -> Connector_PinHeader_2.54mm:PinHeader_1x05_P2.54mm_Horizontal; symbol Connector:Conn_01x04_Socket -> Connector:Conn_01x05_Socket
Connections:
- net col13: now also J4.1 (Pin_1), J5.3 (Pin_3), J6.1 (Pin_1), J8.3 (Pin_3)
- net col14: now also J4.2 (Pin_2), J5.2 (Pin_2), J6.2 (Pin_2), J8.2 (Pin_2)
- net col15: now also J4.3 (Pin_3), J5.1 (Pin_1), J6.3 (Pin_3), J8.1 (Pin_1)
- net col7: no longer J4.1 (Pin_1), J5.1 (Pin_1), J6.1 (Pin_1), J8.1 (Pin_1)
- net col8: no longer J4.2 (Pin_2), J5.2 (Pin_2), J6.2 (Pin_2), J8.2 (Pin_2)
- net col9: no longer J4.3 (Pin_3), J5.3 (Pin_3), J6.3 (Pin_3), J8.3 (Pin_3)
- net row0: now also D_10.1 (K), D_2.1 (K), D_6.1 (K), J3.5 (Pin_5), J7.5 (Pin_5); no longer J3.1 (Pin_1), J7.1 (Pin_1)
- net row1: now also D_11.1 (K), D_3.1 (K), D_7.1 (K), J3.4 (Pin_4), J7.4 (Pin_4); no longer J3.2 (Pin_2), J7.2 (Pin_2)
- net row2: now also D_12.1 (K), D_4.1 (K), D_8.1 (K), J1.4 (Pin_4), J2.4 (Pin_4), J3.2 (Pin_2), J7.2 (Pin_2); no longer J1.3 (Pin_3), J2.3 (Pin_3), J3.3 (Pin_3), J7.3 (Pin_3)
- net row3: now also D_13.1 (K), D_5.1 (K), D_9.1 (K), J1.5 (Pin_5), J2.5 (Pin_5), J3.1 (Pin_1), J7.1 (Pin_1); no longer J1.4 (Pin_4), J2.4 (Pin_4), J3.4 (Pin_4), J7.4 (Pin_4)
- no-connect marks 0 -> 4
Other:
- moved on the sheet: J4, J5, J6, J8

Commit message: Finished
Parts:
- added H1, H2, H3, H4, H5, H6, H7, H8: MountingHole, MountingHole:MountingHole_3.2mm_M3, symbol Mechanical:MountingHole
